File: Small psu.sch (KiCad schematic (older format))
At the start: 39 parts, among them J1 V select sw, J2 VDC-in, J3 reset sw, J4 V out, Q1 BC547, Q2 FQP27P06, U1 LM358, U2 LM317T, U3 LM311N, U4 LM317T, U5 LM358

Commit message: Add files via upload
Parts:
- gave numbers to parts that had none: 1
Connections:
- net GND: no longer U5.2 (-), U5.3 (+)
- net VCC: now also C1.1, J2.1, U2.3 (IN)
- net at J4.2, Q2.2 (S), R11.1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: now also U5.5 (+)
- new net: U5.6 (-), U5.7
Changed lines of the file:
@@
 Connection ~ 3950 2400
 Wire Wire Line
-	3550 2400 3400 2400
+	3400 2400 3550 2400
 Wire Wire Line
 	1200 2400 2600 2400
@@
 	7150 2000 7350 2000
 Wire Wire Line
-	7650 1550 7650 1700
-Wire Wire Line
 	7650 1700 7250 1700
 Wire Wire Line
@@
 	7850 1550 7850 2000
 Wire Wire Line
-	7850 2000 8600 2000
+	7850 2000 9250 2000
 $Comp
 L Screw_Terminal_1x02 J2
@@
 L VCC #PWR021
 U 1 1 5990C98F
-P 2000 2100
-F 0 "#PWR021" H 2000 1950 50  0001 C CNN
-F 1 "VCC" H 2017 2273 50  0000 C CNN
-F 2 "" H 2000 2100 50  0001 C CNN
-F 3 "" H 2000 2100 50  0001 C CNN
-	1    2000 2100
+P 2000 2400
+F 0 "#PWR021" H 2000 2250 50  0001 C CNN
+F 1 "VCC" H 2017 2573 50  0000 C CNN
+F 2 "" H 2000 2400 50  0001 C CNN
+F 3 "" H 2000 2400 50  0001 C CNN
+	1    2000 2400
 	1    0    0    -1
 $EndComp
@@
 Connection ~ 3500 2400
 $Comp
-L LM358 U?
-U 1 1 598EC454
+L LM358 U5
+U 2 1 598EC454
 P 9350 1250
-F 0 "U?" H 9600 1600 50  0000 L CNN
+F 0 "U5" H 9600 1600 50  0000 L CNN
 F 1 "LM358" H 9600 1500 50  0000 L CNN
 F 2 "Housings_DIP:DIP-8_W7.62mm_LongPads" H 9350 1250 50  0001 C CNN
 F 3 "" H 9350 1250 50  0001 C CNN
-	1    9350 1250
+	2    9350 1250
 	0    -1   -1   0
 $EndComp
-$Comp
-L GND #PWR?
-U 1 1 598EC4D8
-P 9250 1550
-F 0 "#PWR?" H 9250 1300 50  0001 C CNN
-F 1 "GND" H 9255 1377 50  0000 C CNN
-F 2 "" H 9250 1550 50  0001 C CNN
-F 3 "" H 9250 1550 50  0001 C CNN
-	1    9250 1550
-	1    0    0    -1
-$EndComp
-$Comp
-L GND #PWR?
-U 1 1 598EC533
-P 9450 1550
-F 0 "#PWR?" H 9450 1300 50  0001 C CNN
-F 1 "GND" H 9455 1377 50  0000 C CNN
-F 2 "" H 9450 1550 50  0001 C CNN
-F 3 "" H 9450 1550 50  0001 C CNN
-	1    9450 1550
-	1    0    0    -1
-$EndComp
-$Comp
-L GND #PWR?
-U 1 1 598EC58E
-P 9350 900
-F 0 "#PWR?" H 9350 650 50  0001 C CNN
-F 1 "GND" H 9355 727 50  0000 C CNN
-F 2 "" H 9350 900 50  0001 C CNN
-F 3 "" H 9350 900 50  0001 C CNN
-	1    9350 900
-	-1   0    0    1
-$EndComp
+Connection ~ 8600 2000
+Connection ~ 7650 1700
+Wire Wire Line
+	7650 1550 7650 1700
+Wire Wire Line
+	9250 2000 9250 1550
+Wire Wire Line
+	9350 950  9350 850
+Wire Wire Line
+	9350 850  9800 850
+Wire Wire Line
+	9800 850  9800 1700
+Wire Wire Line
+	9800 1700 9450 1700
+Wire Wire Line
+	9450 1700 9450 1550
 $EndSCHEMATC

Commit message: Add files via upload
Parts:
- removed U5: LM358, Housings_DIP:DIP-8_W7.62mm_LongPads, symbol LM358
- added U1: LM321, TO_SOT_Packages_SMD:SOT-23-5, symbol LM321
- C1: footprint Capacitors_THT:C_Disc_D3.8mm_W2.6mm_P2.50mm -> Capacitors_SMD:C_0805_HandSoldering
- C2: renamed from C3; footprint Capacitors_THT:CP_Radial_D4.0mm_P2.00mm -> Capacitors_SMD:C_0805_HandSoldering
- C3: renamed from C5; footprint Capacitors_THT:C_Disc_D5.0mm_W2.5mm_P2.50mm -> Capacitors_SMD:C_0805_HandSoldering
- C4: renamed from C2; footprint Capacitors_THT:C_Disc_D3.8mm_W2.6mm_P2.50mm -> Capacitors_SMD:C_0805_HandSoldering
- C5: renamed from C4; footprint Capacitors_THT:C_Disc_D5.0mm_W2.5mm_P2.50mm -> Capacitors_SMD:C_0805_HandSoldering
- C6: footprint Capacitors_THT:C_Disc_D5.0mm_W2.5mm_P2.50mm -> Capacitors_SMD:C_0805_HandSoldering
- D2: renamed from D1; footprint Diodes_THT:D_A-405_P7.62mm_Horizontal -> Diodes_SMD:D_SMA-SMB_Universal_Handsoldering
- D3: renamed from D5; footprint Diodes_THT:D_A-405_P7.62mm_Horizontal -> Diodes_SMD:D_SMA-SMB_Universal_Handsoldering
- Q1: renamed from Q2; footprint TO_SOT_Packages_THT:TO-220_Vertical -> TO_SOT_Packages_THT:TO-220_Horizontal
- R1: renamed from R12; footprint Resistors_THT:R_Axial_DIN0207_L6.3mm_D2.5mm_P7.62mm_Horizontal -> Resistors_SMD:R_0805_HandSoldering
- R10: renamed from R4; footprint Resistors_THT:R_Axial_DIN0207_L6.3mm_D2.5mm_P7.62mm_Horizontal -> Resistors_SMD:R_0805_HandSoldering
- R11: renamed from R10; footprint Resistors_THT:R_Axial_DIN0207_L6.3mm_D2.5mm_P7.62mm_Horizontal -> Resistors_SMD:R_0805_HandSoldering
- R12: renamed from R13; footprint Resistors_THT:R_Axial_DIN0207_L6.3mm_D2.5mm_P7.62mm_Horizontal -> Resistors_SMD:R_0805_HandSoldering
- R13: renamed from R14; footprint Resistors_THT:R_Axial_DIN0207_L6.3mm_D2.5mm_P7.62mm_Horizontal -> Resistors_SMD:R_0805_HandSoldering
- R14: renamed from R1; value 1k6 -> 1k; footprint Resistors_THT:R_Axial_DIN0207_L6.3mm_D2.5mm_P7.62mm_Horizontal -> Resistors_SMD:R_0805_HandSoldering
- R15: renamed from R6; value 1k6 -> 1k; footprint Resistors_THT:R_Axial_DIN0207_L6.3mm_D2.5mm_P7.62mm_Horizontal -> Resistors_SMD:R_0805_HandSoldering
- R2: renamed from R7; footprint Resistors_THT:R_Axial_DIN0207_L6.3mm_D2.5mm_P7.62mm_Horizontal -> Resistors_SMD:R_0805_HandSoldering
- R3: renamed from R8; footprint Resistors_THT:R_Axial_DIN0207_L6.3mm_D2.5mm_P7.62mm_Horizontal -> Resistors_SMD:R_0805_HandSoldering
- R4: renamed from R2; footprint Resistors_THT:R_Axial_DIN0207_L6.3mm_D2.5mm_P7.62mm_Horizontal -> Resistors_THT:R_Axial_DIN0617_L17.0mm_D6.0mm_P20.32mm_Horizontal
- R5: renamed from R15; footprint Resistors_THT:R_Axial_DIN0207_L6.3mm_D2.5mm_P7.62mm_Horizontal -> Resistors_THT:R_Axial_DIN0617_L17.0mm_D6.0mm_P20.32mm_Horizontal
- R6: renamed from R5; footprint Resistors_THT:R_Axial_DIN0207_L6.3mm_D2.5mm_P7.62mm_Horizontal -> Resistors_SMD:R_0805_HandSoldering
- R7: renamed from R9; footprint Resistors_THT:R_Axial_DIN0207_L6.3mm_D2.5mm_P7.62mm_Horizontal -> Resistors_SMD:R_0805_HandSoldering
- R8: renamed from R11; footprint Resistors_THT:R_Axial_DIN0207_L6.3mm_D2.5mm_P7.62mm_Horizontal -> Resistors_SMD:R_0805_HandSoldering
- R9: renamed from R3; footprint Resistors_THT:R_Axial_DIN0207_L6.3mm_D2.5mm_P7.62mm_Horizontal -> Resistors_SMD:R_0805_HandSoldering
- U2: footprint TO_SOT_Packages_THT:TO-220_Vertical -> TO_SOT_Packages_THT:TO-220_Horizontal
- U3: renamed from U4; footprint TO_SOT_Packages_THT:TO-220_Vertical -> TO_SOT_Packages_THT:TO-220_Horizontal
- renumbered D2 to D1, D3 to D4, D4 to D5, J2 to J1, J4 to J2, J1 to J3, J3 to J4, Q1 to Q2, U3 to U4, U1 to U5
Connections:
- net GND: now also U1.2 (V-)
- net VCC: now also U1.5 (V+)
- net at D1.2 (A): now also U1.4
- net at J2.2, Q1.2 (S), R8.1: now also U1.3 (-)
- net at R2.2, R3.1: now also U1.1 (+)
- no-connect marks 1 -> 0
Other:
- note added: "Vin 12vdc"
